File: JL-MP12k.kicad_pcb (KiCad board)
At the start: 4 copper layers, 104.1 x 56.9 mm, 31 parts, among them SW1 RotaryEncoder_Switch, U1 SSD1107

Commit message: fixed some stuff
rev 1.1
Parts:
- added D13: 1N4148W, Diode_SMD:D_SOD-123, B.Cu at (137.2, 88.9)
Connections:
- Gemini1 pad 8: ENC_S1 -> COL4
- SW1 pad S1: ENC_S1 -> Net-(D13-A)
- SW1 pad S2: GND -> COL4
Routing:
- net ENC_S1: track 26.9 -> 0.00 mm
- net COL4: track 0.00 -> 21.9 mm
- net ROW2: track 191.3 -> 206.6 mm
- net Net-(D13-A): track 0.00 -> 13.4 mm
- net 3v3: track 30.3 -> 33.6 mm
- removed copper zone on F.Cu, net GND
Other:
- board size 104.1 x 56.9 mm -> 104.1 x 56.8 mm
- copper layers 4 -> 2
